File: radundant_circuit.kicad_sch (KiCad schematic)
At the start: 15 parts, among them J1 IN1, J2 IN2

Commit message: Autosave
Parts:
- D1: value (none) -> RBQ30NS65ATL

Commit message: Autosave
Parts:
- added D4: 5KPxxA, Diode_THT:D_P600_R-6_P20.00mm_Horizontal, symbol Diode:5KPxxA
Changed lines of the file:
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@@
+	)
+	(symbol
+		(lib_id "Diode:5KPxxA")
+		(at 215.9 85.09 90)
+		(unit 1)
+		(body_style 1)
+		(exclude_from_sim no)
+		(in_bom yes)
+		(on_board yes)
+		(in_pos_files yes)
+		(dnp no)
+		(fields_autoplaced yes)
+		(property "Reference" "D4"
+			(at 218.44 83.8199 90)
+			(show_name no)
+			(do_not_autoplace no)
+			(effects
+				(font
+					(size 1.27 1.27)
+				)
+				(justify right)
+			)
+		)
+		(property "Value" "5KPxxA"
+			(at 218.44 86.3599 90)
+			(show_name no)
+			(do_not_autoplace no)
+			(effects
+				(font
+					(size 1.27 1.27)
+				)
+				(justify right)
+			)
+		)
+		(property "Footprint" "Diode_THT:D_P600_R-6_P20.00mm_Horizontal"
+			(at 220.98 85.09 0)
+			(hide yes)
+			(show_name no)
+			(do_not_autoplace no)
+			(effects
+				(font
+					(size 1.27 1.27)
+				)
+			)
+		)
+		(property "Datasheet" "https://diotec.com/tl_files/diotec/files/pdf/datasheets/5kp65.pdf"
+			(at 215.9 86.36 0)
+			(hide yes)
+			(show_name no)
+			(do_not_autoplace no)
+			(effects
+				(font
+					(size 1.27 1.27)
+				)
+			)
+		)
+		(property "Description" "5000W unidirectional Transient Voltage Suppressor, P-600"
+			(at 215.9 85.09 0)
+			(hide yes)
+			(show_name no)
+			(do_not_autoplace no)
+			(effects
+				(font
+					(size 1.27 1.27)
+				)
+			)
+		)
+		(pin "2"
+		)
+		(pin "1"
+		)
+		(instances
+			(project "radundant_circuit"
+				(path "/2a60c1bb-a3bb-41a5-8345-be72c93980cb"
+					(reference "D4")
+					(unit 1)
+				)
+			)
+		)
 	)
 	(symbol

Commit message: Autosave
Connections:
- net GND: now also D4.1 (A1)
- net OUT: now also D4.2 (A2)
Changed lines of the file:
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@@
+	)
+	(symbol
+		(lib_id "power:GND")
+		(at 215.9 88.9 0)
+		(unit 1)
+		(body_style 1)
+		(exclude_from_sim no)
+		(in_bom yes)
+		(on_board yes)
+		(in_pos_files yes)
+		(dnp no)
+		(fields_autoplaced yes)
+		(property "Reference" "#PWR06"
+			(at 215.9 95.25 0)
+			(hide yes)
+			(show_name no)
+			(do_not_autoplace no)
+			(effects
+				(font
+					(size 1.27 1.27)
+				)
+			)
+		)
+		(property "Value" "GND"
+			(at 215.9 93.98 0)
+			(show_name no)
+			(do_not_autoplace no)
+			(effects
+				(font
+					(size 1.27 1.27)
+				)
+			)
+		)
+		(property "Footprint" ""
+			(at 215.9 88.9 0)
+			(hide yes)
+			(show_name no)
+			(do_not_autoplace no)
+			(effects
+				(font
+					(size 1.27 1.27)
+				)
+			)
+		)
+		(property "Datasheet" ""
+			(at 215.9 88.9 0)
+			(hide yes)
+			(show_name no)
+			(do_not_autoplace no)
+			(effects
+				(font
+					(size 1.27 1.27)
+				)
+			)
+		)
+		(property "Description" "Power symbol creates a global label with name \"GND\" , ground"
+			(at 215.9 88.9 0)
+			(hide yes)
+			(show_name no)
+			(do_not_autoplace no)
+			(effects
+				(font
+					(size 1.27 1.27)
+				)
+			)
+		)
+		(pin "1"
+		)
+		(instances
+			(project "radundant_circuit"
+				(path "/2a60c1bb-a3bb-41a5-8345-be72c93980cb"
+					(reference "#PWR06")
+					(unit 1)
+				)
+			)
+		)
 	)
 	(symbol
@@
 					(unit 1)
 				)
+			)
+		)
+	)
+	(symbol
+		(lib_id "power:+24V")
+		(at 215.9 81.28 0)
+		(unit 1)
+		(body_style 1)
+		(exclude_from_sim no)
+		(in_bom yes)
+		(on_board yes)
+		(in_pos_files yes)
+		(dnp no)
+		(fields_autoplaced yes)
+		(property "Reference" "#PWR_07"
+			(at 215.9 85.09 0)
+			(hide yes)
+			(show_name no)
+			(do_not_autoplace no)
+			(effects
+				(font
+					(size 1.27 1.27)
+				)
+			)
+		)
+		(property "Value" "OUT"
+			(at 215.9 76.2 0)
+			(show_name no)
+			(do_not_autoplace no)
+			(effects
+				(font
+					(size 1.27 1.27)
+				)
+			)
+		)
+		(property "Footprint" ""
+			(at 215.9 81.28 0)
+			(hide yes)
+			(show_name no)
+			(do_not_autoplace no)
+			(effects
+				(font
+					(size 1.27 1.27)
+				)
+			)
+		)
+		(property "Datasheet" ""
+			(at 215.9 81.28 0)
+			(hide yes)
+			(show_name no)
+			(do_not_autoplace no)
+			(effects
+				(font
+					(size 1.27 1.27)
+				)
+			)
+		)
+		(property "Description" "Power symbol creates a global label with name \"+24V\""
+			(at 215.9 81.28 0)
+			(hide yes)
+			(show_name no)
+			(do_not_autoplace no)
+			(effects
+				(font
+					(size 1.27 1.27)
+				)
+			)
+		)
+		(pin "1"
+		)
+		(instances
+			(project "radundant_circuit"
+				(path "/2a60c1bb-a3bb-41a5-8345-be72c93980cb"
+					(reference "#PWR_07")
+					(unit 1)
+				)

Commit message: Autosave
Parts:
- D4: value 5KPxxA -> SMBJ26A; footprint Diode_THT:D_P600_R-6_P20.00mm_Horizontal -> Diode_SMD:D_SMB
Changed lines of the file:
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@@
 			)
 		)
-		(property "Value" "5KPxxA"
+		(property "Value" "SMBJ26A"
 			(at 218.44 86.3599 90)
 			(show_name no)
@@
 			)
 		)
-		(property "Footprint" "Diode_THT:D_P600_R-6_P20.00mm_Horizontal"
+		(property "Footprint" "Diode_SMD:D_SMB"
 			(at 220.98 85.09 0)
 			(hide yes)

Commit message: Autosave
Connections:
- net GND: no longer D4.1 (A1)
- net OUT: no longer D4.2 (A2)
Other:
- moved on the sheet: D4
Changed lines of the file:
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@@
 	(symbol
 		(lib_id "Diode:5KPxxA")
-		(at 215.9 85.09 90)
+		(at 233.68 85.09 270)
 		(unit 1)
 		(body_style 1)
@@
 		(fields_autoplaced yes)
 		(property "Reference" "D4"
-			(at 218.44 83.8199 90)
+			(at 236.22 83.8199 90)
 			(show_name no)
 			(do_not_autoplace no)
@@
 					(size 1.27 1.27)
 				)
-				(justify right)
+				(justify left)
 			)
 		)
 		(property "Value" "SMBJ26A"
-			(at 218.44 86.3599 90)
+			(at 236.22 86.3599 90)
 			(show_name no)
 			(do_not_autoplace no)
@@
 					(size 1.27 1.27)
 				)
-				(justify right)
+				(justify left)
 			)
 		)
 		(property "Footprint" "Diode_SMD:D_SMB"
-			(at 220.98 85.09 0)
+			(at 228.6 85.09 0)
 			(hide yes)
 			(show_name no)
@@
 		)
 		(property "Datasheet" "https://diotec.com/tl_files/diotec/files/pdf/datasheets/5kp65.pdf"
-			(at 215.9 86.36 0)
+			(at 233.68 83.82 0)
 			(hide yes)
 			(show_name no)
@@
 		)
 		(property "Description" "5000W unidirectional Transient Voltage Suppressor, P-600"
-			(at 215.9 85.09 0)
+			(at 233.68 85.09 0)
 			(hide yes)
 			(show_name no)

Commit message: Autosave
Connections:
- net GND: now also D4.2 (A2)
- net OUT: now also D4.1 (A1)
Other:
- moved on the sheet: D4
Changed lines of the file:
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@@
 	(symbol
 		(lib_id "Diode:5KPxxA")
-		(at 233.68 85.09 270)
+		(at 215.9 85.09 270)
 		(unit 1)
 		(body_style 1)
@@
 		(fields_autoplaced yes)
 		(property "Reference" "D4"
-			(at 236.22 83.8199 90)
+			(at 218.44 83.8199 90)
 			(show_name no)
 			(do_not_autoplace no)
@@
 		)
 		(property "Value" "SMBJ26A"
-			(at 236.22 86.3599 90)
+			(at 218.44 86.3599 90)
 			(show_name no)
 			(do_not_autoplace no)
@@
 		)
 		(property "Footprint" "Diode_SMD:D_SMB"
-			(at 228.6 85.09 0)
+			(at 210.82 85.09 0)
 			(hide yes)
 			(show_name no)
@@
 		)
 		(property "Datasheet" "https://diotec.com/tl_files/diotec/files/pdf/datasheets/5kp65.pdf"
-			(at 233.68 83.82 0)
+			(at 215.9 83.82 0)
 			(hide yes)
 			(show_name no)
@@
 		)
 		(property "Description" "5000W unidirectional Transient Voltage Suppressor, P-600"
-			(at 233.68 85.09 0)
+			(at 215.9 85.09 0)
 			(hide yes)
 			(show_name no)

Commit message: Autosave
Parts:
- C2: value C -> 1u
Changed lines of the file:
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@@
 			)
 		)
-		(property "Value" "C"
+		(property "Value" "1u"
 			(at 185.42 87.6299 0)
 			(show_name no)

Commit message: Autosave
Parts:
- C3: value C -> 0.1u
Changed lines of the file:
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@@
 			)
 		)
-		(property "Value" "C"
+		(property "Value" "0.1u"
 			(at 196.85 87.6299 0)
 			(show_name no)
