File: radundant_circuit.kicad_sch (KiCad schematic)
At the start: 16 parts, among them J1 IN1, J2 IN2

Commit message: Autosave
Parts:
- D2, D3: footprint (none) -> LED_SMD:LED_0603_1608Metric_Pad1.05x0.95mm_HandSolder
- F1, F2: footprint (none) -> IMRC_footprint:FUSE_SOCKET
- R1, R2: footprint (none) -> Resistor_SMD:R_0603_1608Metric_Pad0.98x0.95mm_HandSolder
- TP1, TP2, TP3: footprint (none) -> TestPoint:TestPoint_Pad_D1.5mm
Changed lines of the file:
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@@
 			)
 		)
-		(property "Footprint" ""
+		(property "Footprint" "Resistor_SMD:R_0603_1608Metric_Pad0.98x0.95mm_HandSolder"
 			(at 113.792 54.61 90)
 			(hide yes)
@@
 			)
 		)
-		(property "Footprint" ""
+		(property "Footprint" "TestPoint:TestPoint_Pad_D1.5mm"
 			(at 209.55 44.45 0)
 			(hide yes)
@@
 			)
 		)
-		(property "Footprint" ""
+		(property "Footprint" "IMRC_footprint:FUSE_SOCKET"
 			(at 105.41 50.038 90)
 			(hide yes)
@@
 			)
 		)
-		(property "Footprint" ""
+		(property "Footprint" "TestPoint:TestPoint_Pad_D1.5mm"
 			(at 134.62 87.63 0)
 			(hide yes)
@@
 			)
 		)
-		(property "Footprint" ""
+		(property "Footprint" "LED_SMD:LED_0603_1608Metric_Pad1.05x0.95mm_HandSolder"
 			(at 115.57 102.87 0)
 			(hide yes)
@@
 			)
 		)
-		(property "Footprint" ""
+		(property "Footprint" "TestPoint:TestPoint_Pad_D1.5mm"
 			(at 133.35 44.45 0)
 			(hide yes)
@@
 			)
 		)
-		(property "Footprint" ""
+		(property "Footprint" "Resistor_SMD:R_0603_1608Metric_Pad0.98x0.95mm_HandSolder"
 			(at 113.792 95.25 90)
 			(hide yes)
@@
 			)
 		)
-		(property "Footprint" ""
+		(property "Footprint" "LED_SMD:LED_0603_1608Metric_Pad1.05x0.95mm_HandSolder"
 			(at 115.57 62.23 0)
 			(hide yes)
@@
 			)
 		)
-		(property "Footprint" ""
+		(property "Footprint" "IMRC_footprint:FUSE_SOCKET"
 			(at 105.41 93.218 90)
 			(hide yes)

Commit message: SCH Save
Parts:
- TP1: value IN2_TestPoint -> IN1_TestPoint
Changed lines of the file:
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@@
 			)
 		)
-		(property "Value" "IN2_TestPoint"
+		(property "Value" "IN1_TestPoint"
 			(at 130.81 42.4179 0)
 			(show_name no)

Commit message: Autosave
Parts:
- added D5: D, LED_SMD:LED_0603_1608Metric_Pad1.05x0.95mm_HandSolder, symbol Device:D
- added F3: Fuse, IMRC_footprint:FUSE_SOCKET, symbol Device:Fuse
- added J3: IN1, Connector_AMASS:AMASS_XT60-F_1x02_P7.20mm_Vertical, symbol Connector:Conn_01x02_Socket
- added R3: R, Resistor_SMD:R_0603_1608Metric_Pad0.98x0.95mm_HandSolder, symbol Device:R
- added TP4: IN1_TestPoint, TestPoint:TestPoint_Pad_D1.5mm, symbol Connector:TestPoint
Connections:
- net GND: now also D5.1 (K), J3.1 (Pin_1)
- net IN1: now also F3.2, R3.1, TP4.1
- new net: F3.1, J3.2 (Pin_2)
- new net: D5.2 (A), R3.2

Commit message: Autosave
Parts:
- removed F3: Fuse, IMRC_footprint:FUSE_SOCKET, symbol Device:Fuse
Connections:
- net IN1: now also J3.2 (Pin_2)
Other:
- moved on the sheet: D5, R3, TP4
Changed lines of the file:
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@@
 	(paper "A4")
+	(junction
+		(at 185.42 124.46)
+		(diameter 0)
+		(color 0 0 0 0)
+	)
+	(junction
+		(at 184.15 99.06)
+		(diameter 0)
+		(color 0 0 0 0)
+	)
+	(junction
+		(at 115.57 48.26)
+		(diameter 0)
+		(color 0 0 0 0)
+	)
+	(junction
+		(at 198.12 46.99)
+		(diameter 0)
+		(color 0 0 0 0)
+	)
+	(junction
+		(at 124.46 91.44)
+		(diameter 0)
+		(color 0 0 0 0)
+	)
 	(junction
 		(at 193.04 124.46)
@@
 	)
 	(junction
-		(at 184.15 99.06)
-		(diameter 0)
-		(color 0 0 0 0)
-	)
-	(junction
-		(at 115.57 48.26)
-		(diameter 0)
-		(color 0 0 0 0)
-	)
-	(junction
-		(at 198.12 46.99)
-		(diameter 0)
-		(color 0 0 0 0)
-	)
-	(junction
-		(at 124.46 91.44)
-		(diameter 0)
-		(color 0 0 0 0)
-	)
-	(junction
-		(at 200.66 124.46)
-		(diameter 0)
-		(color 0 0 0 0)
-	)
-	(junction
 		(at 167.64 99.06)
 		(diameter 0)
@@
 	(wire
 		(pts
-			(xy 205.74 124.46) (xy 205.74 120.65)
+			(xy 198.12 124.46) (xy 198.12 120.65)
 		)
 		(stroke
@@
 	(wire
 		(pts
-			(xy 205.74 124.46) (xy 200.66 124.46)
+			(xy 198.12 124.46) (xy 193.04 124.46)
 		)
 		(stroke
@@
 	(wire
 		(pts
-			(xy 200.66 119.38) (xy 200.66 124.46)
-		)
-		(stroke
-			(width 0)
-			(type default)
-		)
-	)
-	(wire
-		(pts
-			(xy 186.69 124.46) (xy 193.04 124.46)
+			(xy 193.04 119.38) (xy 193.04 124.46)
 		)
 		(stroke
@@
 	(wire
 		(pts
-			(xy 193.04 124.46) (xy 200.66 124.46)
+			(xy 185.42 124.46) (xy 193.04 124.46)
 		)
 		(stroke
@@
 	(wire
 		(pts
-			(xy 179.07 124.46) (xy 176.53 124.46)
-		)
-		(stroke
-			(width 0)
-			(type default)
-		)
-	)
-	(wire
-		(pts
-			(xy 193.04 127) (xy 193.04 124.46)
+			(xy 176.53 124.46) (xy 185.42 124.46)
+		)
+		(stroke
+			(width 0)
+			(type default)
+		)
+	)
+	(wire
+		(pts
+			(xy 185.42 127) (xy 185.42 124.46)
 		)
 		(stroke
@@
 	(symbol
 		(lib_id "Connector:TestPoint")
-		(at 205.74 120.65 0)
+		(at 198.12 120.65 0)
 		(unit 1)
 		(body_style 1)
@@
 		(fields_autoplaced yes)
 		(property "Reference" "TP4"
-			(at 208.28 116.0779 0)
+			(at 200.66 116.0779 0)
 			(show_name no)
 			(do_not_autoplace no)
@@
 		)
 		(property "Value" "IN1_TestPoint"
-			(at 208.28 118.6179 0)
+			(at 200.66 118.6179 0)
 			(show_name no)
 			(do_not_autoplace no)
@@
 		)
 		(property "Footprint" "TestPoint:TestPoint_Pad_D1.5mm"
-			(at 210.82 120.65 0)
+			(at 203.2 120.65 0)
 			(hide yes)
 			(show_name no)
@@
 		)
 		(property "Datasheet" ""
-			(at 210.82 120.65 0)
+			(at 203.2 120.65 0)
 			(hide yes)
 			(show_name no)
@@
 		)
 		(property "Description" "test point"
-			(at 205.74 120.65 0)
+			(at 198.12 120.65 0)
 			(hide yes)
 			(show_name no)
@@
 	(symbol
 		(lib_id "power:+24V")
-		(at 200.66 119.38 0)
+		(at 193.04 119.38 0)
 		(unit 1)
 		(body_style 1)
@@
 		(fields_autoplaced yes)
 		(property "Reference" "#PWR_08"
-			(at 200.66 123.19 0)
+			(at 193.04 123.19 0)
 			(hide yes)
 			(show_name no)
@@
 		)
 		(property "Value" "IN1"
-			(at 200.66 114.3 0)
+			(at 193.04 114.3 0)
 			(show_name no)
 			(do_not_autoplace no)
@@
 		)
 		(property "Footprint" ""
-			(at 200.66 119.38 0)
+			(at 193.04 119.38 0)
 			(hide yes)
 			(show_name no)
@@
 		)
 		(property "Datasheet" ""
-			(at 200.66 119.38 0)
+			(at 193.04 119.38 0)
 			(hide yes)
 			(show_name no)
@@
 		)
 		(property "Description" "Power symbol creates a global label with name \"+24V\""
-			(at 200.66 119.38 0)
+			(at 193.04 119.38 0)
 			(hide yes)
 			(show_name no)
@@
 	(symbol
 		(lib_id "power:GND")
-		(at 193.04 142.24 0)
+		(at 185.42 142.24 0)
 		(unit 1)
 		(body_style 1)
@@
 		(fields_autoplaced yes)
 		(property "Reference" "#PWR08"
-			(at 193.04 148.59 0)
+			(at 185.42 148.59 0)
 			(hide yes)
 			(show_name no)
@@
 		)
 		(property "Value" "GND"
-			(at 193.04 147.32 0)
+			(at 185.42 147.32 0)
 			(show_name no)
 			(do_not_autoplace no)
@@
 		)
 		(property "Footprint" ""
-			(at 193.04 142.24 0)
+			(at 185.42 142.24 0)
 			(hide yes)
 			(show_name no)
@@
 		)
 		(property "Datasheet" ""
-			(at 193.04 142.24 0)
+			(at 185.42 142.24 0)
 			(hide yes)
 			(show_name no)
@@
 		)
 		(property "Description" "Power symbol creates a global label with name \"GND\" , ground"
-			(at 193.04 142.24 0)
+			(at 185.42 142.24 0)
 			(hide yes)
 			(show_name no)
@@
 	(symbol
 		(lib_id "Device:D")
-		(at 193.04 138.43 90)
+		(at 185.42 138.43 90)
 		(unit 1)
 		(body_style 1)
@@
 		(fields_autoplaced yes)
 		(property "Reference" "D5"
-			(at 195.58 137.1599 90)
+			(at 187.96 137.1599 90)
 			(show_name no)
 			(do_not_autoplace no)
@@
 		)
 		(property "Value" "D"
-			(at 195.58 139.6999 90)
+			(at 187.96 139.6999 90)
 			(show_name no)
 			(do_not_autoplace no)
@@
 		)
 		(property "Footprint" "LED_SMD:LED_0603_1608Metric_Pad1.05x0.95mm_HandSolder"
-			(at 193.04 138.43 0)
+			(at 185.42 138.43 0)
 			(hide yes)
 			(show_name no)
@@
 		)
 		(property "Datasheet" ""
-			(at 193.04 138.43 0)
+			(at 185.42 138.43 0)
 			(hide yes)
 			(show_name no)
@@
 		)
 		(property "Description" "Diode"
-			(at 193.04 138.43 0)
+			(at 185.42 138.43 0)
 			(hide yes)
 			(show_name no)
@@
 		)
 		(property "Sim.Device" "D"
-			(at 193.04 138.43 0)
+			(at 185.42 138.43 0)
 			(hide yes)
 			(show_name no)
@@
 		)
 		(property "Sim.Pins" "1=K 2=A"
-			(at 193.04 138.43 0)
+			(at 185.42 138.43 0)
 			(hide yes)
 			(show_name no)
@@
 	(symbol
 		(lib_id "Device:R")
-		(at 193.04 130.81 0)
+		(at 185.42 130.81 0)
 		(unit 1)
 		(body_style 1)
@@
 		(fields_autoplaced yes)
 		(property "Reference" "R3"
-			(at 195.58 129.5399 0)
+			(at 187.96 129.5399 0)
 			(show_name no)
 			(do_not_autoplace no)
@@
 		)
 		(property "Value" "R"
-			(at 195.58 132.0799 0)
+			(at 187.96 132.0799 0)
 			(show_name no)
 			(do_not_autoplace no)
@@
 		)
 		(property "Footprint" "Resistor_SMD:R_0603_1608Metric_Pad0.98x0.95mm_HandSolder"
-			(at 191.262 130.81 90)
+			(at 183.642 130.81 90)
 			(hide yes)
 			(show_name no)
@@
 		)
 		(property "Datasheet" ""
-			(at 193.04 130.81 0)
+			(at 185.42 130.81 0)
 			(hide yes)
 			(show_name no)
@@
 		)
 		(property "Description" "Resistor"
-			(at 193.04 130.81 0)
+			(at 185.42 130.81 0)
 			(hide yes)
 			(show_name no)
@@
 					(unit 1)
 				)
-			)
-		)
-	)
-	(symbol
-		(lib_id "Device:Fuse")
-		(at 182.88 124.46 90)
-		(unit 1)
-		(body_style 1)
-		(exclude_from_sim no)
-		(in_bom yes)
-		(on_board yes)
-		(in_pos_files yes)
-		(dnp no)
-		(fields_autoplaced yes)
-		(property "Reference" "F3"
-			(at 182.88 118.11 90)
-			(show_name no)
-			(do_not_autoplace no)
-			(effects
-				(font
-					(size 1.27 1.27)
-				)
-			)
-		)
-		(property "Value" "Fuse"
-			(at 182.88 120.65 90)
-			(show_name no)
-			(do_not_autoplace no)
-			(effects
-				(font
-					(size 1.27 1.27)
-				)
-			)
-		)
-		(property "Footprint" "IMRC_footprint:FUSE_SOCKET"
-			(at 182.88 126.238 90)
-			(hide yes)
-			(show_name no)
-			(do_not_autoplace no)
-			(effects
-				(font
-					(size 1.27 1.27)
-				)
-			)
-		)
-		(property "Datasheet" ""
-			(at 182.88 124.46 0)
-			(hide yes)
-			(show_name no)
-			(do_not_autoplace no)
-			(effects
-				(font
-					(size 1.27 1.27)
-				)
-			)
-		)
-		(property "Description" "Fuse"
-			(at 182.88 124.46 0)
-			(hide yes)
-			(show_name no)
-			(do_not_autoplace no)
-			(effects
-				(font
-					(size 1.27 1.27)
-				)
-			)
-		)
-		(pin "1"
-		)
-		(pin "2"
-		)
-		(instances
-			(project "radundant_circuit"
-				(path "/2a60c1bb-a3bb-41a5-8345-be72c93980cb"
-					(reference "F3")
-					(unit 1)
-				)

Commit message: Autosave
Connections:
- net IN1: no longer J3.2 (Pin_2), R3.1, TP4.1
- net OUT: now also J3.2 (Pin_2), R3.1, TP4.1

Commit message: Autosave
Parts:
- removed TP4: IN1_TestPoint, TestPoint:TestPoint_Pad_D1.5mm, symbol Connector:TestPoint
Changed lines of the file:
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@@
-	)
-	(junction
-		(at 193.04 124.46)
-		(diameter 0)
-		(color 0 0 0 0)
 	)
 	(junction
@@
 	(wire
 		(pts
-			(xy 198.12 124.46) (xy 198.12 120.65)
-		)
-		(stroke
-			(width 0)
-			(type default)
-		)
-	)
-	(wire
-		(pts
 			(xy 124.46 91.44) (xy 129.54 91.44)
 		)
@@
 	(wire
 		(pts
-			(xy 198.12 124.46) (xy 193.04 124.46)
-		)
-		(stroke
-			(width 0)
-			(type default)
-		)
-	)
-	(wire
-		(pts
 			(xy 101.6 91.44) (xy 99.06 91.44)
 		)
@@
 		)
 	)
-	(symbol
-		(lib_id "Connector:TestPoint")
-		(at 198.12 120.65 0)
-		(unit 1)
-		(body_style 1)
-		(exclude_from_sim no)
-		(in_bom yes)
-		(on_board yes)
-		(in_pos_files yes)
-		(dnp no)
-		(fields_autoplaced yes)
-		(property "Reference" "TP4"
-			(at 200.66 116.0779 0)
-			(show_name no)
-			(do_not_autoplace no)
-			(effects
-				(font
-					(size 1.27 1.27)
-				)
-				(justify left)
-			)
-		)
-		(property "Value" "IN1_TestPoint"
-			(at 200.66 118.6179 0)
-			(show_name no)
-			(do_not_autoplace no)
-			(effects
-				(font
-					(size 1.27 1.27)
-				)
-				(justify left)
-			)
-		)
-		(property "Footprint" "TestPoint:TestPoint_Pad_D1.5mm"
-			(at 203.2 120.65 0)
-			(hide yes)
-			(show_name no)
-			(do_not_autoplace no)
-			(effects
-				(font
-					(size 1.27 1.27)
-				)
-			)
-		)
-		(property "Datasheet" ""
-			(at 203.2 120.65 0)
-			(hide yes)
-			(show_name no)
-			(do_not_autoplace no)
-			(effects
-				(font
-					(size 1.27 1.27)
-				)
-			)
-		)
-		(property "Description" "test point"
-			(at 198.12 120.65 0)
-			(hide yes)
-			(show_name no)
-			(do_not_autoplace no)
-			(effects
-				(font
-					(size 1.27 1.27)
-				)
-			)
-		)
-		(pin "1"
-		)
-		(instances
-			(project "radundant_circuit"
-				(path "/2a60c1bb-a3bb-41a5-8345-be72c93980cb"
-					(reference "TP4")
-					(unit 1)
-				)
-			)
-		)
-	)

Commit message: SCH Save
Parts:
- J3: value IN1 -> OUT
Changed lines of the file:
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@@
 			)
 		)
-		(property "Value" "IN1"
+		(property "Value" "OUT"
 			(at 172.085 121.92 0)
 			(show_name no)

Commit message: Autosave
Connections:
- net IN2: now also D1.3 (A2); no longer D1.2 (A2)
- net OUT: now also D1.2 (C); no longer D1.3 (C)
