File: radundant_circuit.kicad_pcb (KiCad board)
At the start: 2 copper layers, 19 parts, among them J1 IN1, J2 IN2, J3 OUT

Commit message: Autosave
Parts:
- moved F1 21.0 mm to (65.8, 31.6)
- moved J1 13.6 mm to (50.0, 39.1), turned to 90 degrees
- moved J2 10.3 mm to (50.0, 56.6), turned to 90 degrees
Changed lines of the file:
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@@
 	(footprint "IMRC_footprint:FUSE_SOCKET"
 		(layer "F.Cu")
-		(at 82.9 43.75)
+		(at 65.8 31.575)
 		(property "Reference" "F1"
 			(at 0 -0.75 0)
@@
 	(footprint "Connector_AMASS:AMASS_XT60-F_1x02_P7.20mm_Vertical"
 		(layer "F.Cu")
-		(at 60.175 58.375)
+		(at 50 56.6 90)
 		(descr "AMASS female XT60, through hole, vertical, https://www.tme.eu/Document/2d152ced3b7a446066e6c419d84bb460/XT60%20SPEC.pdf")
 		(tags "XT60 female vertical")
 		(property "Reference" "J2"
-			(at 3.6 -5.3 180)
+			(at 3.6 -5.3 90)
 			(layer "F.SilkS")
 			(effects
@@
 		)
 		(property "Value" "IN2"
-			(at 3.6 5.4 0)
+			(at 3.6 5.4 90)
 			(layer "F.Fab")
 			(effects
@@
 		)
 		(property "Datasheet" ""
-			(at 0 0 0)
+			(at 0 0 90)
 			(unlocked yes)
 			(layer "F.Fab")
@@
 		)
 		(property "Description" "Generic connector, single row, 01x02, script generated"
-			(at 0 0 0)
+			(at 0 0 90)
 			(unlocked yes)
 			(layer "F.Fab")
@@
 		(duplicate_pad_numbers_are_jumpers no)
 		(fp_line
+			(start 11.45 -4.15)
+			(end -1.4 -4.15)
+			(stroke
+				(width 0.12)
+				(type solid)
+			)
+			(layer "F.SilkS")
+		)
+		(fp_line
+			(start -1.4 -4.15)
+			(end -4.25 -1.6)
+			(stroke
+				(width 0.12)
+				(type solid)
+			)
+			(layer "F.SilkS")
+		)
+		(fp_line
 			(start -4.25 -1.6)
 			(end -4.25 1.55)
@@
 		)
 		(fp_line
-			(start -1.4 -4.15)
-			(end -4.25 -1.6)
+			(start 11.45 4.15)
+			(end 11.45 -4.15)
 			(stroke
 				(width 0.12)
@@
 		)
 		(fp_line
-			(start 11.45 -4.15)
-			(end -1.4 -4.15)
-			(stroke
-				(width 0.12)
-				(type solid)
-			)
-			(layer "F.SilkS")
-		)
-		(fp_line
-			(start 11.45 4.15)
-			(end 11.45 -4.15)
-			(stroke
-				(width 0.12)
-				(type solid)
-			)
-			(layer "F.SilkS")
+			(start 11.85 -4.6)
+			(end 11.85 4.6)
+			(stroke
+				(width 0.05)
+				(type solid)
+			)
+			(layer "F.CrtYd")
+		)
+		(fp_line
+			(start -1.6 -4.6)
+			(end 11.85 -4.6)
+			(stroke
+				(width 0.05)
+				(type solid)
+			)
+			(layer "F.CrtYd")
 		)
 		(fp_line
@@
 		)
 		(fp_line
-			(start -1.6 -4.6)
-			(end 11.85 -4.6)
+			(start 11.85 4.6)
+			(end -1.6 4.6)
 			(stroke
 				(width 0.05)
@@
 		)
 		(fp_line
-			(start 11.85 -4.6)
-			(end 11.85 4.6)
-			(stroke
-				(width 0.05)
-				(type solid)
-			)
-			(layer "F.CrtYd")
-		)
-		(fp_line
-			(start 11.85 4.6)
-			(end -1.6 4.6)
-			(stroke
-				(width 0.05)
-				(type solid)
-			)
-			(layer "F.CrtYd")
+			(start 11.35 -4.05)
+			(end -1.4 -4.05)
+			(stroke
+				(width 0.12)
+				(type solid)
+			)
+			(layer "F.Fab")
+		)
+		(fp_line
+			(start -1.4 -4.05)
+			(end -4.15 -1.55)
+			(stroke
+				(width 0.12)
+				(type solid)
+			)
+			(layer "F.Fab")
 		)
 		(fp_line
@@
 		)
 		(fp_line
-			(start -1.4 -4.05)
-			(end -4.15 -1.55)
+			(start 11.35 4.05)
+			(end 11.35 -4.05)
 			(stroke
 				(width 0.12)
@@
 			(layer "F.Fab")
 		)
-		(fp_line
-			(start 11.35 -4.05)
-			(end -1.4 -4.05)
-			(stroke
-				(width 0.12)
-				(type solid)
-			)
-			(layer "F.Fab")
-		)
-		(fp_line
-			(start 11.35 4.05)
-			(end 11.35 -4.05)
-			(stroke
-				(width 0.12)
-				(type solid)
-			)
-			(layer "F.Fab")
-		)
 		(fp_text user "${REFERENCE}"
-			(at 3.6 0.05 0)
+			(at 3.6 0.05 90)
 			(layer "F.Fab")
 			(effects
@@
 		)
 		(pad "1" thru_hole roundrect
-			(at 0 0)
+			(at 0 0 90)
 			(size 6 6)
 			(drill 4.5)
@@
 		)
 		(pad "2" thru_hole circle
-			(at 7.2 0)
+			(at 7.2 0 90)
 			(size 6 6)
 			(drill 4.5)
@@
 	(footprint "Connector_AMASS:AMASS_XT60-F_1x02_P7.20mm_Vertical"
 		(layer "F.Cu")
-		(at 60.175 48.125)
+		(at 50 39.1 90)
 		(descr "AMASS female XT60, through hole, vertical, https://www.tme.eu/Document/2d152ced3b7a446066e6c419d84bb460/XT60%20SPEC.pdf")
 		(tags "XT60 female vertical")
 		(property "Reference" "J1"
-			(at 3.6 -5.3 180)
+			(at 3.6 -5.3 90)
 			(layer "F.SilkS")
 			(effects
@@
 		)
 		(property "Value" "IN1"
-			(at 3.6 5.4 0)
+			(at 3.6 5.4 90)
 			(layer "F.Fab")
 			(effects
@@
 		)
 		(property "Datasheet" ""
-			(at 0 0 0)
+			(at 0 0 90)
 			(unlocked yes)
 			(layer "F.Fab")
@@
 		)
 		(property "Description" "Generic connector, single row, 01x02, script generated"
-			(at 0 0 0)
+			(at 0 0 90)
 			(unlocked yes)
 			(layer "F.Fab")
@@
 		(duplicate_pad_numbers_are_jumpers no)
 		(fp_line
+			(start 11.45 -4.15)
+			(end -1.4 -4.15)
+			(stroke
+				(width 0.12)
+				(type solid)
+			)
+			(layer "F.SilkS")
+		)
+		(fp_line
+			(start -1.4 -4.15)
+			(end -4.25 -1.6)
+			(stroke
+				(width 0.12)
+				(type solid)
+			)
+			(layer "F.SilkS")
+		)
+		(fp_line
 			(start -4.25 -1.6)
 			(end -4.25 1.55)
@@
 		)
 		(fp_line
-			(start -1.4 -4.15)
-			(end -4.25 -1.6)
+			(start 11.45 4.15)
+			(end 11.45 -4.15)
 			(stroke
 				(width 0.12)
@@
 		)
 		(fp_line
-			(start 11.45 -4.15)
-			(end -1.4 -4.15)
-			(stroke
-				(width 0.12)
-				(type solid)
-			)
-			(layer "F.SilkS")
-		)
-		(fp_line
-			(start 11.45 4.15)
-			(end 11.45 -4.15)
-			(stroke
-				(width 0.12)
-				(type solid)
-			)
-			(layer "F.SilkS")
+			(start 11.85 -4.6)
+			(end 11.85 4.6)
+			(stroke
+				(width 0.05)
+				(type solid)
+			)
+			(layer "F.CrtYd")
+		)
+		(fp_line
+			(start -1.6 -4.6)
+			(end 11.85 -4.6)
+			(stroke
+				(width 0.05)
+				(type solid)
+			)
+			(layer "F.CrtYd")
 		)
 		(fp_line
@@
 		)
 		(fp_line
-			(start -1.6 -4.6)
-			(end 11.85 -4.6)
+			(start 11.85 4.6)
+			(end -1.6 4.6)
 			(stroke
 				(width 0.05)
@@
 		)
 		(fp_line
-			(start 11.85 -4.6)
-			(end 11.85 4.6)
-			(stroke
-				(width 0.05)
-				(type solid)
-			)
-			(layer "F.CrtYd")
-		)
-		(fp_line
-			(start 11.85 4.6)
-			(end -1.6 4.6)
-			(stroke
-				(width 0.05)
-				(type solid)
-			)
-			(layer "F.CrtYd")
+			(start 11.35 -4.05)
+			(end -1.4 -4.05)
+			(stroke
+				(width 0.12)
+				(type solid)
+			)
+			(layer "F.Fab")
+		)
+		(fp_line
+			(start -1.4 -4.05)
+			(end -4.15 -1.55)
+			(stroke
+				(width 0.12)
+				(type solid)
+			)
+			(layer "F.Fab")
 		)
 		(fp_line
@@
 		)
 		(fp_line
-			(start -1.4 -4.05)
-			(end -4.15 -1.55)
+			(start 11.35 4.05)
+			(end 11.35 -4.05)
 			(stroke
 				(width 0.12)
@@
 			(layer "F.Fab")
 		)
-		(fp_line
-			(start 11.35 -4.05)
-			(end -1.4 -4.05)
-			(stroke
-				(width 0.12)
-				(type solid)
-			)
-			(layer "F.Fab")
-		)
-		(fp_line
-			(start 11.35 4.05)
-			(end 11.35 -4.05)
-			(stroke
-				(width 0.12)
-				(type solid)
-			)
-			(layer "F.Fab")
-		)
 		(fp_text user "${REFERENCE}"
-			(at 3.6 0.05 0)
+			(at 3.6 0.05 90)
 			(layer "F.Fab")
 			(effects
@@
 		)
 		(pad "1" thru_hole roundrect
-			(at 0 0)
+			(at 0 0 90)
 			(size 6 6)
 			(drill 4.5)
@@
 		)
 		(pad "2" thru_hole circle
-			(at 7.2 0)
+			(at 7.2 0 90)
 			(size 6 6)
 			(drill 4.5)

Commit message: Autosave
Parts:
- moved F2 16.9 mm to (66.3, 49.1)
Changed lines of the file:
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@@
 	(footprint "IMRC_footprint:FUSE_SOCKET"
 		(layer "F.Cu")
-		(at 82.9 52.1)
+		(at 66.3 49.075)
 		(property "Reference" "F2"
 			(at 0 -0.75 0)

Commit message: Autosave
Parts:
- moved J3 54.4 mm to (109.9, 46.5)
- moved TP1 44.1 mm to (78.5, 35.0)
- moved D1 42.2 mm to (89.9, 43.7)
- moved TP2 23.5 mm to (80.0, 65.0)
- moved C1 16.3 mm to (94.5, 64.0)
Changed lines of the file:
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@@
 	(footprint "Package_TO_SOT_SMD:TO-263-2"
 		(layer "F.Cu")
-		(at 83.275 85.425)
+		(at 89.925 43.725)
 		(descr "TO-263/D2PAK/DDPAK SMD package, http://www.infineon.com/cms/en/product/packages/PG-TO263/PG-TO263-3-1/")
 		(tags "D2PAK DDPAK TO-263 D2PAK-3 TO-263-3 SOT-404")
@@
 	(footprint "TestPoint:TestPoint_Pad_D1.5mm"
 		(layer "F.Cu")
-		(at 61.125 75.525)
+		(at 78.5 35)
 		(descr "SMD pad as test Point, diameter 1.5mm")
 		(tags "test point SMD pad")
@@
 	(footprint "Capacitor_THT:CP_Radial_D18.0mm_P7.50mm"
 		(layer "F.Cu")
-		(at 79.11944 69.475)
+		(at 94.52222 64)
 		(descr "CP, Radial series, Radial, pin pitch=7.50mm, diameter=18mm, height=35mm, Electrolytic Capacitor")
 		(tags "CP Radial series Radial pin pitch 7.50mm diameter 18mm height 35mm Electrolytic Capacitor")
@@
 	(footprint "TestPoint:TestPoint_Pad_D1.5mm"
 		(layer "F.Cu")
-		(at 61.125 79.075)
+		(at 80 65)
 		(descr "SMD pad as test Point, diameter 1.5mm")
 		(tags "test point SMD pad")
@@
 	(footprint "Connector_AMASS:AMASS_XT60-F_1x02_P7.20mm_Vertical"
 		(layer "F.Cu")
-		(at 60.175 68.625)
+		(at 109.9 46.5)
 		(descr "AMASS female XT60, through hole, vertical, https://www.tme.eu/Document/2d152ced3b7a446066e6c419d84bb460/XT60%20SPEC.pdf")
 		(tags "XT60 female vertical")

Commit message: Autosave
Parts:
- moved TP2 12.2 mm to (78.0, 53.0)
Changed lines of the file:
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@@
 	(footprint "TestPoint:TestPoint_Pad_D1.5mm"
 		(layer "F.Cu")
-		(at 80 65)
+		(at 78 53)
 		(descr "SMD pad as test Point, diameter 1.5mm")
 		(tags "test point SMD pad")

Commit message: Autosave
Parts:
- moved D1 8.28 mm to (81.7, 44.0)
- moved F2 5.02 mm to (65.8, 54.1)
- moved F1 4.53 mm to (65.3, 27.1)
Changed lines of the file:
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@@
 	(footprint "IMRC_footprint:FUSE_SOCKET"
 		(layer "F.Cu")
-		(at 65.8 31.575)
+		(at 65.3 27.075)
 		(property "Reference" "F1"
 			(at 0 -0.75 0)
@@
 	(footprint "IMRC_footprint:FUSE_SOCKET"
 		(layer "F.Cu")
-		(at 66.3 49.075)
+		(at 65.8 54.075)
 		(property "Reference" "F2"
 			(at 0 -0.75 0)
@@
 	(footprint "Package_TO_SOT_SMD:TO-263-2"
 		(layer "F.Cu")
-		(at 89.925 43.725)
+		(at 81.65 44.04)
 		(descr "TO-263/D2PAK/DDPAK SMD package, http://www.infineon.com/cms/en/product/packages/PG-TO263/PG-TO263-3-1/")
 		(tags "D2PAK DDPAK TO-263 D2PAK-3 TO-263-3 SOT-404")

Commit message: Autosave
Parts:
- moved D1 14.0 mm to (67.7, 44.0)
Changed lines of the file:
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@@
 	(footprint "Package_TO_SOT_SMD:TO-263-2"
 		(layer "F.Cu")
-		(at 81.65 44.04)
+		(at 67.65 44.04)
 		(descr "TO-263/D2PAK/DDPAK SMD package, http://www.infineon.com/cms/en/product/packages/PG-TO263/PG-TO263-3-1/")
 		(tags "D2PAK DDPAK TO-263 D2PAK-3 TO-263-3 SOT-404")

Commit message: Autosave
Parts:
- moved J3 11.6 mm to (98.4, 45.0)
Changed lines of the file:
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@@
 	(footprint "Connector_AMASS:AMASS_XT60-F_1x02_P7.20mm_Vertical"
 		(layer "F.Cu")
-		(at 109.9 46.5)
+		(at 98.4 45)
 		(descr "AMASS female XT60, through hole, vertical, https://www.tme.eu/Document/2d152ced3b7a446066e6c419d84bb460/XT60%20SPEC.pdf")
 		(tags "XT60 female vertical")

Commit message: Autosave
Connections:
- D1 pad 2: IN2 -> OUT
- D1 pad 3: OUT -> IN2
Changed lines of the file:
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@@
 			(unit
 				(name "A")
-				(pins "1" "2" "3")
+				(pins "1" "3" "2")
 			)
 		)
@@
 			(layers "F.Cu" "F.Mask")
 			(roundrect_rratio 0.026596)
-			(net "IN2")
-			(pinfunction "A2_2")
-			(pintype "power_in")
+			(net "OUT")
+			(pinfunction "C_2")
+			(pintype "power_out")
 		)
 		(pad "3" smd roundrect
@@
 			(layers "F.Cu" "F.Mask" "F.Paste")
 			(roundrect_rratio 0.227273)
-			(net "OUT")
-			(pinfunction "C_3")
-			(pintype "power_out")
+			(net "IN2")
+			(pinfunction "A2_3")
+			(pintype "power_in")
 		)
 		(embedded_fonts no)
