File: radundant_circuit.kicad_pcb (KiCad board)
At the start: 2 copper layers, 19 parts, among them J1 IN1, J2 IN2, J3 OUT

Commit message: Autosave
Parts:
- moved F2 1.50 mm to (65.3, 50.6)
- moved F1 0.50 mm to (66.3, 30.6)
Changed lines of the file:
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@@
 	(footprint "IMRC_footprint:FUSE_SOCKET"
 		(layer "F.Cu")
-		(at 66.3 30.075)
+		(at 66.3 30.575)
 		(property "Reference" "F1"
 			(at 0 -0.75 0)
@@
 	(footprint "IMRC_footprint:FUSE_SOCKET"
 		(layer "F.Cu")
-		(at 65.3 52.075)
+		(at 65.3 50.575)
 		(property "Reference" "F2"
 			(at 0 -0.75 0)

Commit message: Autosave
Parts:
- added H1: MountingHole, MountingHole:MountingHole_3.2mm_M3, F.Cu at (31.0, 34.0)
- added H2: MountingHole, MountingHole:MountingHole_3.2mm_M3, F.Cu at (31.0, 41.9)
- added H3: MountingHole, MountingHole:MountingHole_3.2mm_M3, F.Cu at (31.0, 49.9)
- added H4: MountingHole, MountingHole:MountingHole_3.2mm_M3, F.Cu at (31.0, 57.8)

Commit message: Autosave
Parts:
- moved H2 20.5 mm to (43.0, 58.5)
- moved H1 12.5 mm to (43.0, 30.5)
Changed lines of the file:
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@@
 	(footprint "MountingHole:MountingHole_3.2mm_M3"
 		(layer "F.Cu")
-		(at 30.975 33.975)
+		(at 43 30.5)
 		(descr "Mounting Hole 3.2mm, M3, no annular, generated by kicad-footprint-generator mountinghole.py")
 		(tags "mountinghole M3")
@@
 	(footprint "MountingHole:MountingHole_3.2mm_M3"
 		(layer "F.Cu")
-		(at 30.975 41.925)
+		(at 43 58.5)
 		(descr "Mounting Hole 3.2mm, M3, no annular, generated by kicad-footprint-generator mountinghole.py")
 		(tags "mountinghole M3")

Commit message: Autosave
Parts:
- moved H3 72.7 mm to (101.0, 30.5)
- moved H4 70.1 mm to (101.0, 54.5)
Changed lines of the file:
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@@
 	(footprint "MountingHole:MountingHole_3.2mm_M3"
 		(layer "F.Cu")
-		(at 30.975 57.825)
+		(at 101 54.5)
 		(descr "Mounting Hole 3.2mm, M3, no annular, generated by kicad-footprint-generator mountinghole.py")
 		(tags "mountinghole M3")
@@
 	(footprint "MountingHole:MountingHole_3.2mm_M3"
 		(layer "F.Cu")
-		(at 30.975 49.875)
+		(at 101 30.5)
 		(descr "Mounting Hole 3.2mm, M3, no annular, generated by kicad-footprint-generator mountinghole.py")
 		(tags "mountinghole M3")

Commit message: Autosave
Parts:
- moved TP3 11.9 mm to (102.0, 39.5)
Changed lines of the file:
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@@
 	(footprint "TestPoint:TestPoint_Pad_D1.5mm"
 		(layer "F.Cu")
-		(at 113.5 36.5)
+		(at 102 39.5)
 		(descr "SMD pad as test Point, diameter 1.5mm")
 		(tags "test point SMD pad")

Commit message: Autosave
Parts:
- moved C1 1.40 mm to (86.5, 38.0)
Changed lines of the file:
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@@
 	(footprint "Capacitor_THT:CP_Radial_D18.0mm_P7.50mm"
 		(layer "F.Cu")
-		(at 85.52222 39)
+		(at 86.5 38)
 		(descr "CP, Radial series, Radial, pin pitch=7.50mm, diameter=18mm, height=35mm, Electrolytic Capacitor")
 		(tags "CP Radial series Radial pin pitch 7.50mm diameter 18mm height 35mm Electrolytic Capacitor")

Commit message: Autosave
Parts:
- moved D4 22.2 mm to (97.5, 64.5)
Changed lines of the file:
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@@
 	(footprint "Diode_SMD:D_SMB"
 		(layer "F.Cu")
-		(at 116.5 76)
+		(at 97.5 64.5)
 		(descr "Diode SMB (DO-214AA)")
 		(tags "Diode SMB (DO-214AA)")
@@
 		)
 		(property "Value" "SMBJ26A"
-			(at 52.375 -43.025 0)
+			(at -0.5 3.5 0)
 			(layer "F.Fab")
 			(effects

Commit message: Autosave
Parts:
- moved C2 7.72 mm to (81.4, 67.5)
- moved C3 7.72 mm to (81.4, 70.0)
- moved J3 4.40 mm to (96.5, 54.0)
- moved H4 3.50 mm to (104.5, 54.5)
- moved H3 3.04 mm to (104.0, 30.0)
- moved C1 1.50 mm to (88.0, 38.0)
Changed lines of the file:
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@@
 	(footprint "MountingHole:MountingHole_3.2mm_M3"
 		(layer "F.Cu")
-		(at 101 54.5)
+		(at 104.5 54.5)
 		(descr "Mounting Hole 3.2mm, M3, no annular, generated by kicad-footprint-generator mountinghole.py")
 		(tags "mountinghole M3")
@@
 	(footprint "Capacitor_SMD:C_0603_1608Metric_Pad1.08x0.95mm_HandSolder"
 		(layer "F.Cu")
-		(at 87.6375 74.5)
+		(at 81.3625 70)
 		(descr "Capacitor SMD 0603 (1608 Metric), square (rectangular) end terminal, IPC-7351 nominal with elongated pad for handsoldering. (Body size source: IPC-SM-782 page 76, https://www.pcb-3d.com/wordpress/wp-content/uploads/ipc-sm-782a_amendment_1_and_2.pdf)")
 		(tags "capacitor handsolder")
@@
 	(footprint "MountingHole:MountingHole_3.2mm_M3"
 		(layer "F.Cu")
-		(at 101 30.5)
+		(at 104 30)
 		(descr "Mounting Hole 3.2mm, M3, no annular, generated by kicad-footprint-generator mountinghole.py")
 		(tags "mountinghole M3")
@@
 	(footprint "Capacitor_SMD:C_0603_1608Metric_Pad1.08x0.95mm_HandSolder"
 		(layer "F.Cu")
-		(at 87.6375 71.99)
+		(at 81.3625 67.49)
 		(descr "Capacitor SMD 0603 (1608 Metric), square (rectangular) end terminal, IPC-7351 nominal with elongated pad for handsoldering. (Body size source: IPC-SM-782 page 76, https://www.pcb-3d.com/wordpress/wp-content/uploads/ipc-sm-782a_amendment_1_and_2.pdf)")
 		(tags "capacitor handsolder")
@@
 	(footprint "Capacitor_THT:CP_Radial_D18.0mm_P7.50mm"
 		(layer "F.Cu")
-		(at 86.5 38)
+		(at 88 38)
 		(descr "CP, Radial series, Radial, pin pitch=7.50mm, diameter=18mm, height=35mm, Electrolytic Capacitor")
 		(tags "CP Radial series Radial pin pitch 7.50mm diameter 18mm height 35mm Electrolytic Capacitor")
@@
 	(footprint "Connector_AMASS:AMASS_XT60-F_1x02_P7.20mm_Vertical"
 		(layer "F.Cu")
-		(at 92.1 54 180)
+		(at 96.5 54 180)
 		(descr "AMASS female XT60, through hole, vertical, https://www.tme.eu/Document/2d152ced3b7a446066e6c419d84bb460/XT60%20SPEC.pdf")
 		(tags "XT60 female vertical")
